File: KiCad Base Project/Freilab_Blinkies.kicad_sch (KiCad schematic)
At the start: 5 parts, among them SW1 SW_SPDT

Commit message: Added Base Project, restarted PCB layout, added gerbers for base
Signed-off-by: Matteo Hoeren <matteo.hoeren@gmail.com>
Parts:
- D1, D2, D3: footprint LED_THT:LED_D5.0mm_Horizontal_O6.35mm_Z9.0mm -> LED_SMD:BigPad_5mm LED
- SW1: footprint Button_Switch_THT:SW_Slide-03_Wuerth-WS-SLTV_10x2.5x6.4_P2.54mm -> Button_Switch_THT:SW_Toggle_2P1T_5pin
Changed lines of the file:
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@@
 			)
 		)
-		(property "Footprint" "LED_THT:LED_D5.0mm_Horizontal_O6.35mm_Z9.0mm"
+		(property "Footprint" "LED_SMD:BigPad_5mm LED"
 			(at 156.21 83.82 0)
 			(effects
@@
 			)
 		)
-		(property "Footprint" "LED_THT:LED_D5.0mm_Horizontal_O6.35mm_Z9.0mm"
+		(property "Footprint" "LED_SMD:BigPad_5mm LED"
 			(at 156.21 99.06 0)
 			(effects
@@
 			)
 		)
-		(property "Footprint" "LED_THT:LED_D5.0mm_Horizontal_O6.35mm_Z9.0mm"
+		(property "Footprint" "LED_SMD:BigPad_5mm LED"
 			(at 156.21 68.58 0)
 			(effects
@@
 			)
 		)
-		(property "Footprint" "Button_Switch_THT:SW_Slide-03_Wuerth-WS-SLTV_10x2.5x6.4_P2.54mm"
+		(property "Footprint" "Button_Switch_THT:SW_Toggle_2P1T_5pin"
 			(at 154.94 120.65 0)
 			(effects
