File: KiCad Base Project/Freilab_Blinkies.kicad_pcb (KiCad board)
At the start: 2 copper layers, 40 x 40 mm, 11 parts, among them SW1 SW_SPDT

Commit message: Fixed Base DRC Errors, added Tab project & gerbers
Signed-off-by: Matteo Hoeren <matteo.hoeren@gmail.com>
Routing:
- net Net-(BT1--): track 62.0 -> 64.8 mm, vias 1 -> 2
- net Net-(BT1-+): track 24.6 -> 25.5 mm, vias 0 -> 1

Commit message: Added final gerbers for the 3 subprojects
Signed-off-by: Matteo Hoeren <matteo.hoeren@gmail.com>
Parts:
- added ?: , , F.Cu at (210.8, 124.0)
- added ?: , , F.Cu at (180.1, 124.3)
- added ?: , , B.Cu at (210.8, 124.0)
- added ?: , , B.Cu at (180.1, 124.3)
- added ?: , , B.Cu at (195.8, 97.3)
- added REF**: Tab_Pad, MountingEquipment:Tab_Pad, F.Cu at (195.3, 97.3)
- moved REF** 4.47 mm to (196.0, 128.5), turned to 0 degrees
- moved D2 2.55 mm to (187.6, 119.2)
- moved G*** 2.11 mm to (186.3, 122.5)
- moved G*** 1.18 mm to (212.0, 112.9)
Routing:
- net Net-(D1-A): track 53.5 -> 51.5 mm
- net Net-(BT1--): track 64.8 -> 62.8 mm
